File: KICAD/i2v/i2v.kicad_sch (KiCad schematic)
At the start: 32 parts, among them J1 Conn_01x03_Socket, J2 Conn_01x02_Socket, J3 Conn_01x02_Socket, J4 Conn_01x02_Socket, J5 Conn_01x02_Socket, SW1 SW_Rotary_1x6_MP, SW2 SW_Rotary_1x6_MP, U1 NJM2043

Commit message: small fixes in KiCAD and DXF
Parts:
- C2, C3: value 100uF -> 22uF
Changed lines of the file:
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@@
 			)
 		)
-		(property "Value" "100uF"
+		(property "Value" "22uF"
 			(at 92.71 42.2909 0)
 			(show_name no)
@@
 			)
 		)
-		(property "Value" "100uF"
+		(property "Value" "22uF"
 			(at 92.71 57.5309 0)
 			(show_name no)
