File: KICAD/v2i/v2i.kicad_sch (KiCad schematic)
At the start: 31 parts, among them J1 Conn_01x03_Socket, J2 Conn_01x02_Socket, J4 Conn_01x02_Socket, J5 Conn_01x02_Socket, SW1 SW_Rotary_1x6_MP, SW2 SW_Rotary_1x6_MP, U1 NJM2068M

Commit message: small fixes in KiCAD and DXF
Parts:
- C2, C3: value 100uF -> 22uF
